Commit message: Type: Feat Scope: CMake, Package.xml, .cpp, .launch, urdf, rviz Subject: Add VFH & GroundRemove Node for practice. Update build method and rviz as well.

File: urdf/depth_camera.urdf (robot description, URDF)
Before this commit: robot depth_camera, 3 links, 2 joints
Joints:
- joint camera_depth_joint: origin xyz=0 0 0 rpy=0 1.57 0 -> xyz=0 0 0 rpy=0 0 0
- joint camera_joint: origin xyz=0 0 0 rpy=0 0 0 -> xyz=0 0 0 rpy=3.14159 0 0

Commit message: Fix point cloud coordinate issue.

File: urdf/depth_camera.urdf (robot description, URDF)
Before this commit: robot depth_camera, 3 links, 2 joints
Joints:
- joint camera_depth_joint: origin xyz=0 0 0 rpy=0 0 0 -> xyz=0 0 0 rpy=0 0 3.1415926
- joint camera_joint: origin xyz=0 0 0 rpy=3.14159 0 0 -> xyz=0 0 0 rpy=0 0 0
